Commit message: feat: multi-format map loading, auto .bt cache, world_loader library
- octo_planner now supports .pcd/.bt/.ot/.world/.sdf with automatic
  extension detection and corresponding loaders
- Auto-save .bt cache after first conversion; subsequent loads skip
  conversion when cache is newer than source (auto_save_bt=true)
- New world_loader library: tinyxml2-based SDF parser + geometry
  voxelization ported from jie_3d_nav world_to_octomap_node
- New maps/npz_to_bt.py: convert jie_3d_nav NPZ maps to .bt format
- New params: auto_save_bt, world_xy_window_size_m
- Simulation: 3D LiDAR publishes PointCloud2 natively (/lidar_points),
  localPlanner remaps /registered_scan → /lidar_points
- Docs: consolidate map format details in quickstart, simplify other docs

Co-Authored-By: Claude Opus 4.7 <noreply@anthropic.com>

File: src/simulation/urdf/diff_drive_robot.urdf.xacro (robot description, xacro)
@@ -156,5 +156,5 @@
     <origin xyz="${-base_length/2 + 0.05} 0 ${-base_z_offset + caster_radius}" rpy="0 0 0"/>
   </joint>
-  <!-- Lidar Link (for obstacle detection topic compatibility) -->
+  <!-- 3D LiDAR (mimics real robot dog: front-mounted, 10° downward pitch) -->
   <link name="lidar_link">
     <visual>
@@ -172,5 +172,5 @@
     <parent link="base_link"/>
     <child link="lidar_link"/>
-    <origin xyz="0 0 ${base_height/2 + 0.025}" rpy="0 0 0"/>
+    <origin xyz="${base_length/2} 0 ${base_height/2 + 0.025}" rpy="0 0.174533 0"/>
   </joint>
   <!-- Gazebo Plugins -->
@@ -208,7 +208,7 @@
     </plugin>
   </gazebo>
-  <!-- 2D Lidar for obstacle awareness -->
+  <!-- 3D LiDAR: 360° HFOV, -7°~52° VFOV, 10Hz, PointCloud2 output -->
   <gazebo reference="lidar_link">
-    <sensor type="ray" name="lidar">
+    <sensor type="gpu_ray" name="lidar_3d">
       <pose>0 0 0 0 0 0</pose>
       <visualize>false</visualize>
@@ -222,16 +222,21 @@
             <max_angle>3.14159</max_angle>
           </horizontal>
+          <vertical>
+            <samples>20</samples>
+            <min_angle>-0.122173</min_angle>
+            <max_angle>0.907571</max_angle>
+          </vertical>
         </scan>
         <range>
           <min>0.15</min>
-          <max>8.0</max>
+          <max>30.0</max>
           <resolution>0.01</resolution>
         </range>
       </ray>
-      <plugin name="scan" filename="libgazebo_ros_ray_sensor.so">
+      <plugin name="lidar_3d_plugin" filename="libgazebo_ros_ray_sensor.so">
         <ros>
-          <remapping>~/out:=scan</remapping>
+          <remapping>~/out:=lidar_points</remapping>
         </ros>
-        <output_type>sensor_msgs/LaserScan</output_type>
+        <output_type>sensor_msgs/PointCloud2</output_type>
         <frame_name>lidar_link</frame_name>
       </plugin>
