Commit message: feat: simulation SLAM closed-loop + non-avoidance navigation + controller fixes
Simulation ↔ real-robot alignment (A1 mode):
- URDF: remove base_footprint / imu_link / lidar_link; base_link is root
- LiDAR+IMU on trunk, frame=livox_frame, topics /livox/lidar /livox/imu
- LiDAR pose: x=+0.15 front, z=+0.13 above, pitch=-15° matching real robot
- LiDAR density: 720×28 = 20,160 pts/scan (~Livox Mid-360 200k pts/s)
- A1RLController: publish_odom / publish_tf SDF params for SLAM mode
- gazebo.launch.py: slam_mode param; non-SLAM static TFs; xacro arg injection
- slam.launch.py: update static TF to match new LiDAR position
- Car LiDAR density synced to match

Non-avoidance navigation (skip latticePlanner):
- pathFollower: use_global_path mode subscribing to /planned_path
- TF-based map→base_link transform, waypoint management (lookahead,
  advance, rear-guard, goal detection), pure pursuit
- navigation_no_avoidance.launch.py: octo_planner + pathFollower only
- Subscribe to both /path and /planned_path (ROS 2 params after ctor)

Controller fixes (global-path mode):
- Fix sign: dirDiff = -atan2(y,x) so -gain*dirDiff turns toward target
- Skip path-age timeout for global path (replans at 1.5s, not 100Hz)
- noRotAtGoal kept for local-path mode only

Docs & scripts:
- CLAUDE.md, architecture.md, development.md: 3 startup modes documented
- scripts/: slam_mode / use_sim_time / no_avoidance params added

Co-Authored-By: Claude <noreply@anthropic.com>

File: src/simulation/urdf/a1/a1.urdf.xacro (robot description, xacro)
@@ -5,7 +5,5 @@
     <xacro:include filename="$(find simulation)/urdf/a1/leg.xacro"/>
     <xacro:include filename="$(find simulation)/urdf/a1/gazebo.xacro"/>
-    <!-- Root link (matching car convention) -->
-    <link name="base_footprint"/>
-    <!-- Robot base link (matches car convention: base_footprint → base_link) -->
+    <!-- Root: base_link (matches real robot — no base_footprint). -->
     <link name="base_link">
         <visual>
@@ -16,9 +14,4 @@
         </visual>
     </link>
-    <joint name="base_footprint_joint" type="fixed">
-        <parent link="base_footprint"/>
-        <child link="base_link"/>
-        <origin rpy="0 0 0" xyz="0 0 0"/>
-    </joint>
     <!-- Floating base: connects base_link to physical trunk -->
     <joint name="floating_base" type="fixed">
@@ -35,4 +28,12 @@
             </geometry>
             <material name="orange"/>
+        </visual>
+        <!-- LiDAR body visual (pure decoration, not in TF tree) -->
+        <visual>
+            <origin rpy="0 0.261799 0" xyz="0.10 0 0.08"/>
+            <geometry>
+                <mesh filename="$(env A1_MESHES_DIR)/livox_mid360.dae" scale="1 1 1"/>
+            </geometry>
+            <material name="grey"/>
         </visual>
         <collision>
@@ -51,48 +52,7 @@
         </inertial>
     </link>
-    <!-- IMU fixed to trunk center -->
-    <joint name="imu_joint" type="fixed">
-        <parent link="trunk"/>
-        <child link="imu_link"/>
-        <origin rpy="0 0 0" xyz="0 0 0"/>
-    </joint>
-    <link name="imu_link">
-        <inertial>
-            <mass value="0.001"/>
-            <origin rpy="0 0 0" xyz="0 0 0"/>
-            <inertia ixx="0.0001" ixy="0" ixz="0" iyy="0.0001" iyz="0" izz="0.0001"/>
-        </inertial>
-        <visual>
-            <origin rpy="0 0 0" xyz="0 0 0"/>
-            <geometry>
-                <box size="0.001 0.001 0.001"/>
-            </geometry>
-            <material name="red"/>
-        </visual>
-        <collision>
-            <origin rpy="0 0 0" xyz="0 0 0"/>
-            <geometry>
-                <box size=".001 .001 .001"/>
-            </geometry>
-        </collision>
-    </link>
-    <!-- 3D LiDAR: front-mounted on trunk, 10° downward pitch -->
-    <joint name="lidar_joint" type="fixed">
-        <parent link="trunk"/>
-        <child link="lidar_link"/>
-        <origin xyz="0.22 0 0.08" rpy="0 0.174533 0"/>
-    </joint>
-    <link name="lidar_link">
-        <visual>
-            <geometry>
-                <cylinder radius="0.04" length="0.03"/>
-            </geometry>
-            <material name="grey"/>
-        </visual>
-        <inertial>
-            <mass value="0.1"/>
-            <inertia ixx="0.0001" ixy="0" ixz="0" iyy="0.0001" iyz="0" izz="0.0001"/>
-        </inertial>
-    </link>
+    <!-- LiDAR & IMU: NOT in URDF tree — Gazebo plugins attach directly to trunk
+         in gazebo.xacro, publishing in livox_frame. The TF livox_frame ↔ base_link
+         is provided externally (slam.launch.py or gazebo launch static TF). -->
     <!-- Four legs -->
     <xacro:leg name="FR" mirror="-1" mirror_dae="False" front_hind="1" front_hind_dae="True">

File: src/simulation/urdf/a1/gazebo.xacro (robot description, xacro)
@@ -1,4 +1,6 @@
 <?xml version="1.0"?>
 <robot xmlns:xacro="http://www.ros.org/wiki/xacro">
+    <xacro:arg name="publish_odom" default="true"/>
+    <xacro:arg name="publish_tf" default="true"/>
     <!-- A1 RL Controller Plugin: handles 12-DOF locomotion + odom + joint_states + TF -->
     <gazebo>
@@ -26,12 +28,18 @@
             <!-- cmd_vel timeout: zero velocity if no message received (default 0.5s) -->
             <cmdVelTimeout>0.5</cmdVelTimeout>
-            <!-- TF frames -->
+            <!-- TF frames (base_link = root, matches real robot) -->
             <odomFrameId>odom</odomFrameId>
-            <robotBaseFrame>base_footprint</robotBaseFrame>
+            <robotBaseFrame>base_link</robotBaseFrame>
+            <!-- When slam_mode, set these false so SLAM provides odom + TF -->
+            <publish_odom>$(arg publish_odom)</publish_odom>
+            <publish_tf>$(arg publish_tf)</publish_tf>
         </plugin>
     </gazebo>
-    <!-- IMU on trunk -->
-    <gazebo reference="imu_link">
+    <!-- IMU attached directly to trunk, publishes in livox_frame (matches real robot).
+         Position: co-located with LiDAR at x=+0.15 front, z=+0.13 above base_link,
+         pitch=-15° down.  SLAM extrinsic lidar→imu is trivial (~5 cm); ignored in sim. -->
+    <gazebo reference="trunk">
         <sensor type="imu" name="trunk_imu">
+            <pose>0.10 0 0.08 0 0.261799 0</pose>
             <always_on>true</always_on>
             <update_rate>1000</update_rate>
@@ -81,15 +89,16 @@
             <plugin name="trunk_imu_plugin" filename="libgazebo_ros_imu_sensor.so">
                 <ros>
-                    <remapping>~/out:=trunk_imu</remapping>
+                    <remapping>~/out:=livox/imu</remapping>
                 </ros>
                 <initial_orientation_as_reference>false</initial_orientation_as_reference>
-                <frame_name>imu_link</frame_name>
+                <frame_name>livox_frame</frame_name>
             </plugin>
         </sensor>
     </gazebo>
-    <!-- 3D LiDAR (front-mounted, 10° downward pitch, same config as car) -->
-    <gazebo reference="lidar_link">
+    <!-- 3D LiDAR attached to trunk (x=+0.15 front, z=+0.13 above, pitch=-15° down).
+         Matches real-robot livox_frame → base_link static TF in slam.launch.py. -->
+    <gazebo reference="trunk">
         <sensor type="gpu_ray" name="lidar_3d">
-            <pose>0 0 0 0 0 0</pose>
+            <pose>0.10 0 0.08 0 0.261799 0</pose>
             <visualize>false</visualize>
             <update_rate>10</update_rate>
@@ -97,5 +106,5 @@
                 <scan>
                     <horizontal>
-                        <samples>360</samples>
+                        <samples>720</samples>
                         <resolution>1</resolution>
                         <min_angle>-3.14159</min_angle>
@@ -103,5 +112,5 @@
                     </horizontal>
                     <vertical>
-                        <samples>20</samples>
+                        <samples>28</samples>
                         <min_angle>-0.122173</min_angle>
                         <max_angle>0.907571</max_angle>
@@ -116,8 +125,8 @@
             <plugin name="lidar_3d_plugin" filename="libgazebo_ros_ray_sensor.so">
                 <ros>
-                    <remapping>~/out:=lidar_points</remapping>
+                    <remapping>~/out:=livox/lidar</remapping>
                 </ros>
                 <output_type>sensor_msgs/PointCloud2</output_type>
-                <frame_name>lidar_link</frame_name>
+                <frame_name>livox_frame</frame_name>
             </plugin>
         </sensor>

File: src/simulation/urdf/diff_drive_robot.urdf.xacro (robot description, xacro)
@@ -218,5 +218,5 @@
         <scan>
           <horizontal>
-            <samples>360</samples>
+            <samples>720</samples>
             <resolution>1</resolution>
             <min_angle>-3.14159</min_angle>
@@ -224,5 +224,5 @@
           </horizontal>
           <vertical>
-            <samples>20</samples>
+            <samples>28</samples>
             <min_angle>-0.122173</min_angle>
             <max_angle>0.907571</max_angle>
